Commit message: Add files via upload

File: waiter_robot_1/urdf/waiter_robot_1.urdf.xacro (robot description, xacro)
@@ -3,5 +3,7 @@
      Commit Version: 1.6.0-4-g7f85cfe  Build Version: 1.6.7995.38578
      For more information, please see http://wiki.ros.org/sw_urdf_exporter -->
-<robot  name="waiter_robot_1" >
+<robot  name="waiter_robot_1" xmlns:xacro="http://ros.org/wiki/xacro">
+  <xacro:include filename="$(find waiter_robot_1)/urdf/waiter_common_properties.xacro"/>
+  <xacro:include filename="$(find waiter_robot_1)/urdf/waiter_robot_1.gazebo.xacro"/>
   <link name="base_footprint"/>
   <joint name="base_joint" type="fixed">
@@ -361,3 +363,9 @@
   </joint>
   <link name="base_scan"/>
+  <joint name="camera_joint" type="fixed">
+    <parent link="base_link"/>
+    <child link="camera_link"/>
+    <origin xyz="0.16 0.005 0.165" rpy="0 0 0"/>
+  </joint>
+  <link name="camera_link"/>
 </robot>

File: waiter_robot_1/urdf/waiter_robot_1_tf_hoverboard.urdf (robot description, URDF)
Before this commit: robot waiter_robot_1, 10 links, 9 joints
Joints:
- removed joint wheel_left_joint
- removed joint wheel_right_joint
- added joint left_wheel: type continuous, parent base_link, child wheel_left_link, origin xyz=-0.075 0.1942 -0.0125 rpy=-1.5708 0 0, axis 0 0 1
- added joint right_wheel: type continuous, parent base_link, child wheel_right_link, origin xyz=-0.075 -0.1942 -0.0125 rpy=1.5708 0 3.1416, axis 0 0 1
- joint base_joint: origin xyz=0.0 0.0 0.0 rpy=0 0 0 -> xyz=0.0 0.0 0.01 rpy=0 0 0
